File: Hardware/EDA/Arduino_Tau_mikroBUS.sch (KiCad schematic (older format))
At the start: 30 parts, among them J1 HEADER_F_2.54MM_1R8P_ST_AU_PTH, J2 HEADER_F_2.54MM_1R8P_ST_AU_PTH, J3 HEADER_F_2.54MM_1R11P_ST_AU_P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, J4 HEADER_F_2.54MM_1R11P_ST_AU_P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, J5 Molex_0475710001, M1 FID, M2 FID, M3 FID, P1 HEADER_M_2.54MM_1R4P_ST_AU_PTH, P2 HEADER_M_2.54MM_1R4P_ST_AU_PTH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

Commit message: Final changes prior to gerber verification.
Other:
- moved on the sheet: P1, P2, P3, P4, R1, R2
